File: Kicad/PCR.sch (KiCad schematic (older format))
At the start: 52 parts, among them J1 54819-0519, U1 74HCT04, U2 MCP100-450DI, Y1 6.25MHz/30pF

Commit message: Update to work with mostly the default KiCAD items or items downloaded via the KiCAD Libraries too.
2 Resistors added of 1k on the lines for TRUE and FALSE pull ups.

Several things deleted which appeared at Graphic shapes on the PCB sometimes
but could not be edited. this was done manually at the bottom of the PCB_KiCAD file.

Deleted some PCB items around the order which marked the Copper limits of top and bottom. may have been tied to TRUE & FALSE.

Changed USB socket type.

This has been done not to change the board but to aid understanding and allow anyone who wants slightly easier access.

I have not tested it and provide no warranty.

Signed-off-by: John Bradley <flypie@rocketmail.com>
Parts:
- added H1, H2, H3, H4: MountingHole, MountingHole:MountingHole_2.7mm_M2.5, symbol Mechanical:MountingHole
- added R100, R101: 1K, Resistor_THT:R_Axial_DIN0204_L3.6mm_D1.6mm_P1.90mm_Vertical, symbol Device:R
- added unit 7 of U1
- added U11: 74HCT139, Package_DIP:DIP-16_W7.62mm, symbol 74xx:74LS139
- added U16: 74HCT32, Package_DIP:DIP-14_W7.62mm, symbol 74xx:74LS32
- C1, C2, C3: footprint Capacitors_THT:C_Disc_D3.0mm_W2.0mm_P2.50mm -> Capacitor_THT:C_Disc_D3.0mm_W2.0mm_P2.50mm
- C10, C11, C12, C13, C14, C15, C16, C17, C18, C19, C20, C21, C22, C23, C24, C25, C26, C27, C28, C29, C30, C31, C32, C33, C34, C35, C36, C37, C38, C39, C40, C41, C42, C5, C6, C7, C8, C9: footprint Capacitors_THT:C_Disc_D4.3mm_W1.9mm_P5.00mm -> Capacitor_THT:C_Disc_D4.3mm_W1.9mm_P5.00mm
- C4: footprint Capacitors_THT:CP_Radial_D8.0mm_P3.50mm -> Capacitor_THT:CP_Radial_D8.0mm_P3.50mm
- D1: footprint Diodes_THT:D_DO-15_P12.70mm_Horizontal -> Diode_THT:D_DO-15_P12.70mm_Horizontal
- D2: footprint LEDs:LED_D3.0mm -> LED_THT:LED_D3.0mm
- F1: value 750mA/180mΩ/60V -> 750mA/180mohms/60V; footprint Fuse_Holders_and_Fuses:Fuse_TE5_Littlefuse-395Series -> Fuse:Fuse_Littelfuse_395Series
- J1: footprint 54819-0519-MvK:54819-0519-MvK -> Connector_USB:USB_Micro-B_Wuerth_629105150521; symbol Connector:USB_B_Mini -> Connector:USB_B
- R1, R2, R3: footprint Resistors_THT:R_Axial_DIN0207_L6.3mm_D2.5mm_P10.16mm_Horizontal -> Resistor_THT:R_Axial_DIN0207_L6.3mm_D2.5mm_P10.16mm_Horizontal
- U2: footprint TO_SOT_Packages_THT:TO-92_Inline_Wide -> Package_TO_SOT_THT:TO-92L_Inline_Wide
- Y1: footprint Crystals:Crystal_HC49-U_Vertical -> Crystal:Crystal_HC49-U_Vertical
Connections:
- wire segments 198 -> 204
- no-connect marks 4 -> 3
Other:
- moved on the sheet: U2
