File: Kicad/PER.sch (KiCad schematic (older format))
At the start: 23 parts, among them J2 CONN-JACK-STEREO-R/A-3PIN-3.5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, J3 DB15_FEMALE_HighDensity_Mount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, J4 DB9_MALE_MountingHoles, U38 74HCT273, U39 74HC595

Commit message: Update to work with mostly the default KiCAD items or items downloaded via the KiCAD Libraries too.
2 Resistors added of 1k on the lines for TRUE and FALSE pull ups.

Several things deleted which appeared at Graphic shapes on the PCB sometimes
but could not be edited. this was done manually at the bottom of the PCB_KiCAD file.

Deleted some PCB items around the order which marked the Copper limits of top and bottom. may have been tied to TRUE & FALSE.

Changed USB socket type.

This has been done not to change the board but to aid understanding and allow anyone who wants slightly easier access.

I have not tested it and provide no warranty.

Signed-off-by: John Bradley <flypie@rocketmail.com>
Parts:
- C43, C44: footprint Capacitors_THT:C_Disc_D4.3mm_W1.9mm_P5.00mm -> Capacitor_THT:C_Disc_D4.3mm_W1.9mm_P5.00mm
- D5, D6, D7, D8: footprint LEDs:LED_D3.0mm -> LED_THT:LED_D3.0mm
- J2: footprint Kicad:SJ1-3523N-MvK -> SamacSys_Parts_l:SJ13523N; symbol Connector:AudioJack4_Ground -> SamacSys_Parts:SJ1-3523N
- J3: footprint Connector_Dsub:DSUB-15-HD_Female_Vertical_P2.29x1.98mm_MountingHoles -> Connector_Dsub:DSUB-15-HD_Female_Horizontal_P2.29x1.98mm_EdgePinOffset3.03mm_Housed_MountingHolesOffset4.94mm
- J4: footprint Connectors:DB9MD -> Connector_Dsub:DSUB-9_Female_Horizontal_P2.77x2.84mm_EdgePinOffset4.94mm_Housed_MountingHolesOffset7.48mm
- R10, R11, R12, R13, R14, R15, R16, R17, R18, R19: footprint Resistors_THT:R_Axial_DIN0207_L6.3mm_D2.5mm_P10.16mm_Horizontal -> Resistor_THT:R_Axial_DIN0207_L6.3mm_D2.5mm_P10.16mm_Horizontal
- R8: footprint Resistors_THT:R_Array_SIP5 -> Resistor_THT:R_Array_SIP5
- R9: value R=10kΩ -> R=10kohms; footprint Resistors_THT:R_Array_SIP6 -> Resistor_THT:R_Array_SIP6; symbol Gigatron-parts:4606X-R2R-103LF -> SamacSys_Parts:4606X-R2R-103LF
Connections:
- wire segments 135 -> 138
Other:
- note added: "The RGB resistor values depend on the 74xx sub-family of the OUT register:\n 7400/74LS: 390ohms / 820Ω\n 74HCT/HC: 750Ω / 1500Ω"
- note removed: "The RGB resistor values depend on the 74xx sub-family of the OUT register:\n 7400/74LS: 390Ω / 820Ω\n 74HCT/HC: 750Ω / 1500Ω"
- moved on the sheet: C43, C44, R10
