File: Kicad/PRG.sch (KiCad schematic (older format))
At the start: 8 parts, among them U10 74HCT244, U3 74HCT161, U4 74HCT161, U5 74HCT161, U6 74HCT161, U7 27C1024, U8 74HCT273, U9 74HCT273

Commit message: Update to work with mostly the default KiCAD items or items downloaded via the KiCAD Libraries too.
2 Resistors added of 1k on the lines for TRUE and FALSE pull ups.

Several things deleted which appeared at Graphic shapes on the PCB sometimes
but could not be edited. this was done manually at the bottom of the PCB_KiCAD file.

Deleted some PCB items around the order which marked the Copper limits of top and bottom. may have been tied to TRUE & FALSE.

Changed USB socket type.

This has been done not to change the board but to aid understanding and allow anyone who wants slightly easier access.

I have not tested it and provide no warranty.

Signed-off-by: John Bradley <flypie@rocketmail.com>
Parts:
- U7: symbol Gigatron-parts:27C1024 -> SamacSys_Parts:AT27C1024-45PU
Connections:
- net labels added: VCC
- wire segments 190 -> 197
Other:
- moved on the sheet: U10, U3, U4, U5, U6, U8, U9
